File: oresat-c3-card/oresat-c3-sch-osd3358-usb-xtal.kicad_sch (KiCad schematic)
At the start: 38 parts, among them U1 OSD3358-1G-ISM, U11 RCLAMP0504FB, Y1 ECS-240-12-30BQ-AEN-TR, Y2 ABS07-32.768KHZ-T

Commit message: Updating BOM and switching to oresat-passive footprints. Fixed some power cutoff limits, and fixed another DC voltage leverl on an LNA!
Parts:
- C30, C32, U1, U11, Y1, Y2: DST Digi-Key -> DigiKey
- R47: footprint Resistor_SMD:R_0603_1608Metric -> oresat-passives:0603-C-NOSILK; DST Digi-Key -> DigiKey
- R75, R76, R77: footprint Resistor_SMD:R_0603_1608Metric -> oresat-passives:0603-C-NOSILK; DST Digi-Key -> DigiKey; MFR Stackpole Electronics Inc -> Stackpole Electronics
Changed lines of the file:
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@@
 			)
 		)
-		(property "Datasheet" "~"
+		(property "Datasheet" "https://ecsxtal.com/store/pdf/ECX-53BQ.pdf"
 			(at 166.37 81.28 0)
 			(effects
@@
 			)
 		)
-		(property "Description" "Four pin crystal, GND on pins 2 and 4"
+		(property "Description" "CRYSTAL 24.0000MHZ 12PF SMD"
 			(at 166.37 81.28 0)
 			(effects
@@
 			)
 		)
-		(property "DST" "Digi-Key"
+		(property "DST" "DigiKey"
 			(at 166.37 81.28 0)
 			(effects
@@
 			)
 		)
-		(property "DST" "Digi-Key"
+		(property "DST" "DigiKey"
 			(at 167.64 111.76 0)
 			(effects
@@
 			)
 		)
-		(property "Footprint" "Resistor_SMD:R_0603_1608Metric"
+		(property "Footprint" "oresat-passives:0603-C-NOSILK"
 			(at 166.37 138.43 0)
 			(effects
@@
 			)
 		)
-		(property "Datasheet" "~"
+		(property "Datasheet" "https://www.seielect.com/catalog/SEI-RMCF_RMCP.pdf"
 			(at 166.37 138.43 0)
 			(effects
@@
 			)
 		)
-		(property "DST" "Digi-Key"
+		(property "DST" "DigiKey"
 			(at 166.37 138.43 0)
 			(effects
@@
 			)
 		)
-		(property "MFR" "Stackpole Electronics Inc"
+		(property "MFR" "Stackpole Electronics"
 			(at 166.37 138.43 0)
 			(effects
@@
 			)
 		)
-		(property "DST" "Digi-Key"
+		(property "DST" "DigiKey"
 			(at 200.66 207.01 0)
 			(effects
@@
 			)
 		)
-		(property "DST" "Digi-Key"
+		(property "DST" "DigiKey"
 			(at 215.9 196.85 0)
 			(effects
@@
 			)
 		)
-		(property "Datasheet" ""
+		(property "Datasheet" "https://octavosystems.com/docs/osd335x-sm-datasheet/"
 			(at 226.06 116.84 0)
 			(effects
@@
 			)
 		)
-		(property "DST" "Digi-Key"
+		(property "DST" "DigiKey"
 			(at 226.06 116.84 0)
 			(effects
@@
 			)
 		)
-		(property "DST" "Digi-Key"
+		(property "DST" "DigiKey"
 			(at 265.43 91.44 0)
 			(effects
@@
 			)
 		)
-		(property "Footprint" "Resistor_SMD:R_0603_1608Metric"
+		(property "Footprint" "oresat-passives:0603-C-NOSILK"
 			(at 171.45 138.43 0)
 			(effects
@@
 			)
 		)
-		(property "Datasheet" "~"
+		(property "Datasheet" "https://www.seielect.com/catalog/SEI-RMCF_RMCP.pdf"
 			(at 171.45 138.43 0)
 			(effects
@@
 			)
 		)
-		(property "DST" "Digi-Key"
+		(property "DST" "DigiKey"
 			(at 171.45 138.43 0)
 			(effects
@@
 			)
 		)
-		(property "MFR" "Stackpole Electronics Inc"
+		(property "MFR" "Stackpole Electronics"
 			(at 171.45 138.43 0)
 			(effects
@@
 			)
 		)
-		(property "Footprint" "Resistor_SMD:R_0603_1608Metric"
+		(property "Footprint" "oresat-passives:0603-C-NOSILK"
 			(at 180.34 81.28 0)
 			(effects
@@
 			)
 		)
-		(property "Datasheet" "~"
+		(property "Datasheet" "https://www.seielect.com/catalog/SEI-RMCF_RMCP.pdf"
 			(at 180.34 81.28 0)
 			(effects
@@
 			)
 		)
-		(property "DST" "Digi-Key"
+		(property "DST" "DigiKey"
 			(at 180.34 81.28 0)
 			(effects
@@
 			)
 		)
-		(property "Footprint" "Resistor_SMD:R_0603_1608Metric"
+		(property "Footprint" "oresat-passives:0603-C-NOSILK"
 			(at 158.75 148.59 0)
 			(effects
@@
 			)
 		)
-		(property "Datasheet" "~"
+		(property "Datasheet" "https://www.seielect.com/catalog/SEI-RMCF_RMCP.pdf"
 			(at 158.75 148.59 0)
 			(effects
@@
 			)
 		)
-		(property "DST" "Digi-Key"
+		(property "DST" "DigiKey"
 			(at 158.75 148.59 0)
 			(effects
@@
 			)
 		)
-		(property "MFR" "Stackpole Electronics Inc"
+		(property "MFR" "Stackpole Electronics"
 			(at 158.75 148.59 0)
 			(effects

Commit message: All footprints updated. Passes ERC/DRC.
Parts:
- C26, C27: footprint Capacitor_SMD:C_0603_1608Metric -> oresat-passives:0603-C-NOSILK; DPN 399-6840-1-ND -> 399-16015-1-ND; DST Digi-Key -> DigiKey; MPN C0603C100J5GACAUTO -> C0603C100J1GACAUTO
- C28, C29: footprint Capacitor_SMD:C_0603_1608Metric -> oresat-passives:0603-C-NOSILK
- C30, C32: footprint Capacitor_SMD:C_0603_1608Metric -> oresat-passives:0603-C-NOSILK; DPN 587-3472-1-ND -> 399-6856-1-ND; MFR Taiyo Yuden -> KEMET; MPN TMK107BJ104KAHT -> C0603C104K5RACAUTO
- C31: footprint Capacitor_SMD:C_0603_1608Metric -> oresat-passives:0603-C-NOSILK; DPN 399-C0603C102J5GECAUTOCT-ND -> 399-12989-1-ND; DST Digi-Key -> DigiKey; MPN C0603C102J5GECAUTO -> C0603C102J5RACAUTO
Changed lines of the file:
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@@
 			)
 		)
-		(property "Footprint" "Capacitor_SMD:C_0603_1608Metric"
+		(property "Footprint" "oresat-passives:0603-C-NOSILK"
 			(at 153.67 88.9 0)
 			(effects
@@
 			)
 		)
-		(property "Datasheet" "~"
+		(property "Datasheet" "https://www.yageogroup.com/content/datasheet/asset/file/KEM_C1022_C0G_AUTO_SMD"
 			(at 153.67 88.9 0)
 			(effects
@@
 			)
 		)
-		(property "Description" "10pF ±5% 50V Ceramic Capacitor C0G, NP0 0603 (1608 Metric)"
+		(property "Description" "10 pF ±5% 100V Ceramic Capacitor C0G, NP0 0603 (1608 Metric)"
 			(at 153.67 88.9 0)
 			(effects
@@
 			)
 		)
-		(property "DPN" "399-6840-1-ND"
+		(property "DPN" "399-16015-1-ND"
 			(at 153.67 88.9 0)
 			(effects
@@
 			)
 		)
-		(property "DST" "Digi-Key"
+		(property "DST" "DigiKey"
 			(at 153.67 88.9 0)
 			(effects
@@
 			)
 		)
-		(property "MPN" "C0603C100J5GACAUTO"
+		(property "MPN" "C0603C100J1GACAUTO"
 			(at 153.67 88.9 0)
 			(effects
@@
 			)
 		)
-		(property "Footprint" "Capacitor_SMD:C_0603_1608Metric"
+		(property "Footprint" "oresat-passives:0603-C-NOSILK"
 			(at 215.9 196.85 0)
 			(effects
@@
 			)
 		)
-		(property "Datasheet" "~"
+		(property "Datasheet" "https://search.kemet.com/download/specsheet/C0603C104K5RACAUTO"
 			(at 215.9 196.85 0)
 			(effects
@@
 			)
 		)
-		(property "Description" "100 nF (0.1µF) ±10% 25V Ceramic Capacitor X5R 0603 (1608 Metric)"
+		(property "Description" "0.1 µF ±10% 50V Ceramic Capacitor X7R 0603 (1608 Metric)"
 			(at 215.9 196.85 0)
 			(effects
@@
 			)
 		)
-		(property "DPN" "587-3472-1-ND"
+		(property "DPN" "399-6856-1-ND"
 			(at 215.9 196.85 0)
 			(effects
@@
 			)
 		)
-		(property "MFR" "Taiyo Yuden"
+		(property "MFR" "KEMET"
 			(at 215.9 196.85 0)
 			(effects
@@
 			)
 		)
-		(property "MPN" "TMK107BJ104KAHT"
+		(property "MPN" "C0603C104K5RACAUTO"
 			(at 215.9 196.85 0)
 			(effects
@@
 			)
 		)
-		(property "Footprint" "Capacitor_SMD:C_0603_1608Metric"
+		(property "Footprint" "oresat-passives:0603-C-NOSILK"
 			(at 160.02 119.38 0)
 			(effects
@@
 			)
 		)
-		(property "Footprint" "Capacitor_SMD:C_0603_1608Metric"
+		(property "Footprint" "oresat-passives:0603-C-NOSILK"
 			(at 160.02 104.14 0)
 			(effects
@@
 			)
 		)
-		(property "Footprint" "Capacitor_SMD:C_0603_1608Metric"
+		(property "Footprint" "oresat-passives:0603-C-NOSILK"
 			(at 257.81 91.44 0)
 			(effects
@@
 			)
 		)
-		(property "Datasheet" "~"
+		(property "Datasheet" "https://www.yageogroup.com/content/datasheet/asset/file/KEM_C1023_X7R_AUTO_SMD"
 			(at 257.81 91.44 0)
 			(effects
@@
 			)
 		)
-		(property "Description" "1 nF (1000 pF) ±5% 50V Ceramic Capacitor C0G, NP0 0603 (1608 Metric)"
+		(property "Description" "1000 pF ±5% 50V Ceramic Capacitor X7R 0603 (1608 Metric)"
 			(at 257.81 91.44 0)
 			(effects
@@
 			)
 		)
-		(property "DPN" "399-C0603C102J5GECAUTOCT-ND"
+		(property "DPN" "399-12989-1-ND"
 			(at 257.81 91.44 0)
 			(effects
@@
 			)
 		)
-		(property "DST" "Digi-Key"
+		(property "DST" "DigiKey"
 			(at 257.81 91.44 0)
 			(effects
@@
 			)
 		)
-		(property "MPN" "C0603C102J5GECAUTO"
+		(property "MPN" "C0603C102J5RACAUTO"
 			(at 257.81 91.44 0)
 			(effects
@@
 			)
 		)
-		(property "Footprint" "Capacitor_SMD:C_0603_1608Metric"
+		(property "Footprint" "oresat-passives:0603-C-NOSILK"
 			(at 265.43 91.44 0)
 			(effects
@@
 			)
 		)
-		(property "Datasheet" "~"
+		(property "Datasheet" "https://search.kemet.com/download/specsheet/C0603C104K5RACAUTO"
 			(at 265.43 91.44 0)
 			(effects
@@
 			)
 		)
-		(property "Description" "100 nF (0.1µF) ±10% 25V Ceramic Capacitor X5R 0603 (1608 Metric)"
+		(property "Description" "0.1 µF ±10% 50V Ceramic Capacitor X7R 0603 (1608 Metric)"
 			(at 265.43 91.44 0)
 			(effects
@@
 			)
 		)
-		(property "DPN" "587-3472-1-ND"
+		(property "DPN" "399-6856-1-ND"
 			(at 265.43 91.44 0)
 			(effects
@@
 			)
 		)
-		(property "MFR" "Taiyo Yuden"
+		(property "MFR" "KEMET"
 			(at 265.43 91.44 0)
 			(effects
@@
 			)
 		)
-		(property "MPN" "TMK107BJ104KAHT"
+		(property "MPN" "C0603C104K5RACAUTO"
 			(at 265.43 91.44 0)
 			(effects
@@
 			)
 		)
-		(property "Footprint" "Capacitor_SMD:C_0603_1608Metric"
+		(property "Footprint" "oresat-passives:0603-C-NOSILK"
 			(at 153.67 73.66 0)
 			(effects
@@
 			)
 		)
-		(property "Datasheet" "~"
+		(property "Datasheet" "https://www.yageogroup.com/content/datasheet/asset/file/KEM_C1022_C0G_AUTO_SMD"
 			(at 153.67 73.66 0)
 			(effects
@@
 			)
 		)
-		(property "Description" "10pF ±5% 50V Ceramic Capacitor C0G, NP0 0603 (1608 Metric)"
+		(property "Description" "10 pF ±5% 100V Ceramic Capacitor C0G, NP0 0603 (1608 Metric)"
 			(at 153.67 73.66 0)
 			(effects
@@
 			)
 		)
-		(property "DPN" "399-6840-1-ND"
+		(property "DPN" "399-16015-1-ND"
 			(at 153.67 73.66 0)
 			(effects
@@
 			)
 		)
-		(property "DST" "Digi-Key"
+		(property "DST" "DigiKey"
 			(at 153.67 73.66 0)
 			(effects
@@
 			)
 		)
-		(property "MPN" "C0603C100J5GACAUTO"
+		(property "MPN" "C0603C100J1GACAUTO"
 			(at 153.67 73.66 0)
 			(effects
