File: oresat-c3-card/oresat-c3-sch-uhf-band.kicad_sch (KiCad schematic)
At the start: 124 parts, among them Q3 DMP2035UQ-7, Q4 DMN3028LQ-7, U18 LT5534, U19 BDCN-20-13+, U20 QPC1022, U21 TQP7M9105, U22 LT5534, U25 SN74LVC1G11IDCKRQ1, U26 TLV7041DBV, U27 SN74LVC1G04DCKR, U29 TQP3M9036, U32 SF2446E, U33 SF2446E, U40 MAX941EUA+, U44 AT86RF215, U45 NCS2-62+, U47 QPC1022, X3 TXETALSANF-26.000000

Commit message: Changed WDT tantalums to space-rated tantalums (fun) and fixed some BOM issues. Also possibly more silk screen cleanup.
Parts:
- C118, C119, C120, C55, C58, C59, C66, C67, C69, C71, C83, C84, C86, C96: DST Digi-Key -> DigiKey
Changed lines of the file:
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@@
 			)
 		)
-		(property "DST" "Digi-Key"
+		(property "DST" "DigiKey"
 			(at 204.47 105.41 0)
 			(effects
@@
 			)
 		)
-		(property "DST" "Digi-Key"
+		(property "DST" "DigiKey"
 			(at 383.54 38.1 0)
 			(effects
@@
 			)
 		)
-		(property "DST" "Digi-Key"
+		(property "DST" "DigiKey"
 			(at 383.54 55.88 0)
 			(effects
@@
 			)
 		)
-		(property "DST" "Digi-Key"
+		(property "DST" "DigiKey"
 			(at 241.3 55.88 0)
 			(effects
@@
 			)
 		)
-		(property "DST" "Digi-Key"
+		(property "DST" "DigiKey"
 			(at 238.76 104.14 0)
 			(effects
@@
 			)
 		)
-		(property "DST" "Digi-Key"
+		(property "DST" "DigiKey"
 			(at 288.29 224.79 0)
 			(effects
@@
 			)
 		)
-		(property "DST" "Digi-Key"
+		(property "DST" "DigiKey"
 			(at 290.83 128.27 0)
 			(effects
@@
 			)
 		)
-		(property "DST" "Digi-Key"
+		(property "DST" "DigiKey"
 			(at 251.46 224.79 0)
 			(effects
@@
 			)
 		)
-		(property "DST" "Digi-Key"
+		(property "DST" "DigiKey"
 			(at 118.11 128.27 0)
 			(effects
@@
 			)
 		)
-		(property "DST" "Digi-Key"
+		(property "DST" "DigiKey"
 			(at 267.97 55.88 0)
 			(effects
@@
 			)
 		)
-		(property "DST" "Digi-Key"
+		(property "DST" "DigiKey"
 			(at 240.03 38.1 0)
 			(effects
@@
 			)
 		)
-		(property "DST" "Digi-Key"
+		(property "DST" "DigiKey"
 			(at 233.68 100.33 0)
 			(effects
@@
 			)
 		)
-		(property "DST" "Digi-Key"
+		(property "DST" "DigiKey"
 			(at 355.6 55.88 0)
 			(effects
@@
 			)
 		)
-		(property "DST" "Digi-Key"
+		(property "DST" "DigiKey"
 			(at 252.73 212.09 0)
 			(effects

Commit message: Removed unecessary L band 5th order filter. Moved UHF to 401/436 variants
Parts:
- removed U32, U33: SF2446E, oresat-ics:SM3030-6, symbol oresat-ics:SF2446E
- added FL1, FL2: RF1419D, Filter:Filter_SAW-8_3.8x3.8mm, symbol oresat-passives:856930
- C55: footprint oresat-passives:0603-C-NOSILK -> oresat-passives:0402-B-NOSILK; DPN 1276-6566-1-ND -> 490-17515-1-ND; MFR Samsung Electro-Mechanics -> Murata; MPN CL10C8R2CB81PNC -> GCQ1555C1H8R2BB01D
- C85, C87: value 3p -> 3.9p; DPN 490-17461-1-ND -> 490-GCQ1555C1H3R9WB01DCT-ND; MPN GCQ1555C1H3R0CB01D -> GCQ1555C1H3R9WB01D
- C86: value 8.3p -> 8.2p; DPN 399-16122-1-ND -> 490-17515-1-ND; MFR KEMET -> Murata; MPN CBR04C839B5GAC -> GCQ1555C1H8R2BB01D
Connections:
- net GND: now also FL1.1 (GND), FL1.3 (GND), FL1.4 (GND), FL1.5 (GND), FL1.7 (GND), FL1.8 (GND), FL2.1 (GND), FL2.3 (GND), FL2.4 (GND), FL2.5 (GND), FL2.7 (GND), FL2.8 (GND)
- net at TP904.1, U20.8 (RF2): now also FL2.2 (IN)
- net at C118.1, TP906.1: now also FL2.6 (OUT)
- net at C119.2, TP907.1: now also FL1.2 (IN)
- net at TP902.1, U47.4 (RF1): now also FL1.6 (OUT)
Other:
- note added: "5th order LPF for harmonics (F3dB = 600 MHz)"
- note added: "70 cm amateur radio band is 430 - 440 MHz"
- note added: "Alt: TST TA0692A for 436.5 MHz but must be hand placed"
- note added: "For 401 MHz"
- note removed: "5th order LPF for 436.5 MHz"

Commit message: BOM only change: Upgraded single gate inverter to AEC qualified version
Parts:
- FL1, FL2: DST (none) -> DigiKey
- U27: DPN 296-11600-1-ND -> 296-22895-1-ND; MPN SN74LVC1G04DCKR -> SN74LVC1G04QDCKRQ1
Changed lines of the file:
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@@
 			)
 		)
-		(property "Datasheet" "https://www.ti.com/lit/ds/symlink/sn74lvc1g04.pdf"
+		(property "Datasheet" "https://www.ti.com/lit/ds/symlink/sn74lvc1g04.pdf?ts=1753305682684&ref_url=https%253A%252F%252Fwww.ti.com%252Fproduct%252FSN74LVC1G04"
 			(at 127 171.45 0)
 			(effects
@@
 			)
 		)
-		(property "Description" "Single NOT Gate, Low-Voltage CMOS"
+		(property "Description" "Inverter IC 1 Channel SC-70-5"
 			(at 127 171.45 0)
 			(effects
@@
 			)
 		)
-		(property "DPN" "296-11600-1-ND"
+		(property "DPN" "296-22895-1-ND"
 			(at 127 171.45 0)
 			(effects
@@
 			)
 		)
-		(property "MPN" "SN74LVC1G04DCKR"
+		(property "MPN" "SN74LVC1G04QDCKRQ1"
 			(at 127 171.45 0)
 			(effects
@@
 			)
 		)
+		(property "DST" "DigiKey"
+			(at 213.36 224.79 0)
+			(effects
+				(font
+					(size 1.27 1.27)
+				)
+				(hide yes)
+			)
+		)
 		(pin "8"
 		)
@@
 			(at 321.31 224.79 0)
 			(effects
+				(font
+					(size 1.27 1.27)
+				)
+				(hide yes)
+			)
+		)
+		(property "DST" "DigiKey"
+			(at 321.31 224.79 0)
+			(effects
