File: oresat-c3-card/oresat-c3-sch-osd3358-sip-e-f.kicad_sch (KiCad schematic)
At the start: 5 parts, among them U1 OSD3358-1G-ISM

Commit message: Design review on power and RF
Parts:
- U1: Distributor (none) -> DigiKey; MPN OSD3358-1G-ISM -> OSD3358-512M-BSM
Changed lines of the file:
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@@
 			)
 		)
-		(property "Description" "Embedded Module ARM® Cortex®-A8, AM3358 1GHz 1GB"
+		(property "Description" "OSD335x Embedded Module 1GHz 512MB"
 			(at 218.44 78.74 0)
 			(effects
@@
 			)
 		)
-		(property "MPN" "OSD3358-1G-ISM"
+		(property "MPN" "OSD3358-512M-BSM"
 			(at 218.44 83.82 0)
 			(effects
@@
 		(property "MFR" "Octavo Systems"
 			(at 218.44 182.88 0)
+			(effects
+				(font
+					(size 1.27 1.27)
+				)
+				(hide yes)
+			)
+		)
+		(property "Distributor" "DigiKey"
+			(at 218.44 81.28 0)
 			(effects
 				(font
@@
 			)
 		)
-		(property "Description" "Embedded Module ARM® Cortex®-A8, AM3358 1GHz 1GB"
+		(property "Description" "OSD335x Embedded Module 1GHz 512MB"
 			(at 217.17 -16.51 0)
 			(effects
@@
 			)
 		)
-		(property "MPN" "OSD3358-1G-ISM"
+		(property "MPN" "OSD3358-512M-BSM"
 			(at 217.17 -11.43 0)
 			(effects
@@
 			(effects
 				(font
+					(size 1.27 1.27)
+				)
+				(hide yes)
+			)
+		)
+		(property "Distributor" "DigiKey"
+			(at 217.17 -13.97 0)
+			(effects
+				(font

Commit message: Updating BOM and switching to oresat-passive footprints. Fixed some power cutoff limits, and fixed another DC voltage leverl on an LNA!
Parts:
- U1: DST Digi-Key -> DigiKey
Changed lines of the file:
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@@
 			)
 		)
-		(property "Datasheet" ""
+		(property "Datasheet" "https://octavosystems.com/docs/osd335x-sm-datasheet/"
 			(at 218.44 182.88 0)
 			(effects
@@
 			)
 		)
-		(property "DST" "Digi-Key"
+		(property "DST" "DigiKey"
 			(at 218.44 182.88 0)
 			(effects
@@
 			)
 		)
-		(property "Datasheet" ""
+		(property "Datasheet" "https://octavosystems.com/docs/osd335x-sm-datasheet/"
 			(at 217.17 87.63 0)
 			(effects
@@
 			)
 		)
-		(property "DST" "Digi-Key"
+		(property "DST" "DigiKey"
 			(at 217.17 87.63 0)
 			(effects
