File: oresat-c3-card/oresat-c3-sch-osd3358-sysboot.kicad_sch (KiCad schematic)
At the start: 24 parts, among them J6 Conn_01x02, Q2 DMN3028LQ-7, U1 OSD3358-1G-ISM, U39 TCAN330

Commit message: Changed to hierarchy view
Updated schematic to hierarchy view, replaced couple of footprints on pcb and schematic symbols. Deleted connectors sheet.
Changed lines of the file:
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@@
 		)
 	)
-	(global_label "LBAND_LO_nSEN"
-		(shape output)
-		(at 143.51 128.27 180)
-		(fields_autoplaced yes)
+	(hierarchical_label "CAN2_L"
+		(shape input)
+		(at 194.31 91.44 0)
+		(effects
+			(font
+				(size 1.27 1.27)
+			)
+			(justify left)
+		)
+	)
+	(hierarchical_label "CAN2_H"
+		(shape input)
+		(at 194.31 86.36 0)
+		(effects
+			(font
+				(size 1.27 1.27)
+			)
+			(justify left)
+		)
+	)
+	(hierarchical_label "LBAND_LO_SCLK"
+		(shape input)
+		(at 143.51 130.81 180)
 		(effects
 			(font
@@
 			(justify right)
 		)
-		(property "Intersheetrefs" "${INTERSHEET_REFS}"
-			(at 125.4852 128.27 0)
-			(show_name no)
-			(do_not_autoplace no)
-			(effects
-				(font
-					(size 1.27 1.27)
-				)
-				(justify right)
+	)
+	(hierarchical_label "LBAND_LO_nSEN"
+		(shape input)
+		(at 143.51 128.27 180)
+		(effects
+			(font
+				(size 1.27 1.27)
 			)
+			(justify right)
 		)
 	)
-	(global_label "CAN2_L"
-		(shape input)
-		(at 194.31 91.44 0)
-		(fields_autoplaced yes)
+	(hierarchical_label "RADIO_ENABLE"
+		(shape output)
+		(at 229.87 173.99 0)
 		(effects
 			(font
@@
 			(justify left)
 		)
-		(property "Intersheetrefs" "${INTERSHEET_REFS}"
-			(at 204.1895 91.44 0)
-			(show_name no)
-			(do_not_autoplace no)
-			(effects
-				(font
-					(size 1.27 1.27)
-				)
-				(justify left)
-			)
-		)
 	)
-	(global_label "LBAND_LO_SDATA"
-		(shape output)
+	(hierarchical_label "LBAND_LO_SDATA"
+		(shape input)
 		(at 143.51 133.35 180)
-		(fields_autoplaced yes)
 		(effects
 			(font
@@
 			(justify right)
 		)
-		(property "Intersheetrefs" "${INTERSHEET_REFS}"
-			(at 124.6989 133.35 0)
-			(show_name no)
-			(do_not_autoplace no)
-			(effects
-				(font
-					(size 1.27 1.27)
-				)
-				(justify right)
-			)
-		)
 	)
-	(global_label "LBAND_LO_nLOCKED"
+	(hierarchical_label "LBAND_LO_nLOCKED"
 		(shape input)
 		(at 144.78 171.45 180)
-		(fields_autoplaced yes)
 		(effects
 			(font
@@
 			(justify right)
 		)
-		(property "Intersheetrefs" "${INTERSHEET_REFS}"
-			(at 123.1266 171.45 0)
-			(show_name no)
-			(do_not_autoplace no)
-			(effects
-				(font
-					(size 1.27 1.27)
-				)
-				(justify right)
-			)
-		)
 	)
-	(global_label "LBAND_LO_SCLK"
-		(shape output)
-		(at 143.51 130.81 180)
-		(fields_autoplaced yes)
-		(effects
-			(font
-				(size 1.27 1.27)
-			)
-			(justify right)
-		)
-		(property "Intersheetrefs" "${INTERSHEET_REFS}"
-			(at 125.5456 130.81 0)
-			(show_name no)
-			(do_not_autoplace no)
-			(effects
-				(font
-					(size 1.27 1.27)
-				)
-				(justify right)
-			)
-		)
-	)
-	(global_label "PET_WDT"
+	(hierarchical_label "PET_WDT"
 		(shape output)
 		(at 229.87 179.07 0)
-		(fields_autoplaced yes)
 		(effects
 			(font
@@
 			(justify left)
 		)
-		(property "Intersheetrefs" "${INTERSHEET_REFS}"
-			(at 240.819 179.07 0)
-			(show_name no)
-			(do_not_autoplace no)
-			(effects
-				(font
-					(size 1.27 1.27)
-				)
-				(justify left)
-			)
-		)
 	)
-	(global_label "CAN2_H"
-		(shape input)
-		(at 194.31 86.36 0)
-		(fields_autoplaced yes)
-		(effects
-			(font
-				(size 1.27 1.27)
-			)
-			(justify left)
-		)
-		(property "Intersheetrefs" "${INTERSHEET_REFS}"
-			(at 204.4919 86.36 0)
-			(show_name no)
-			(do_not_autoplace no)
-			(effects
-				(font
-					(size 1.27 1.27)
-				)
-				(justify left)
-			)
-		)
-	)
-	(global_label "RADIO_ENABLE"
-		(shape output)
-		(at 229.87 173.99 0)
-		(fields_autoplaced yes)
-		(effects
-			(font
-				(size 1.27 1.27)
-			)
-			(justify left)
-		)
-		(property "Intersheetrefs" "${INTERSHEET_REFS}"
-			(at 246.3225 173.99 0)
-			(show_name no)
-			(do_not_autoplace no)
-			(effects
-				(font
-					(size 1.27 1.27)
-				)
-				(justify left)
-			)
-		)
-	)
