File: oresat-c3-card/oresat-c3.kicad_sch (KiCad schematic)
At the start: 0 parts

Commit message: Changed to hierarchy view
Updated schematic to hierarchy view, replaced couple of footprints on pcb and schematic symbols. Deleted connectors sheet.
Parts:
- added FID1, FID2, FID3: Fiducial, Fiducial:Fiducial_1mm_Mask2mm, symbol Mechanical:Fiducial
- added J1: TFM-120-01-L-D-RA, oresat-connectors:J-SAMTEC-TFM-120-X1-XXX-D-RA, symbol oresat-connectors:J-SAMTEC-TFM-120-01-L-D-RA
- added J3, J4: 2477330-1, oresat-connectors:J-MOLEX-SMPM-073300-002X, symbol oresat-connectors:J-MOLEX-SMPM-73300-002X
- added J7: GRPB041VWVN-RC, Connector_PinHeader_1.27mm:PinHeader_1x04_P1.27mm_Vertical, symbol Connector_Generic:Conn_01x04
- added J8: SM14B-SHLS-TF, oresat-connectors:J-JST-SM14BSHLSTF, symbol oresat-connectors:ORESAT-DEBUG-CONNECTOR-3
- added PCB1: ORESAT-CARD-V1.3-GENERIC-1RF-POS2, oresat-pcbs:ORESAT-CARD-V1.3-2RF-RIGHT, symbol oresat-pcbs:ORESAT-CARD-V1.3-2RF-RIGHT
- added R48: 75, oresat-passives:0603-C-NOSILK, symbol Device:R_Small_US
- added TP106, TP142, TP143, TP144, TP145, TP146, TP147, TP152, TP153, TP154, TP155, TP29, TP30: Test-Point, oresat-misc:TestPoint_Pad_D1.0mm, symbol oresat-misc:Test-Point-1mm-round
Connections:
- new net: J1.6, TP147.1
- new net: J1.1, TP142.1
- new net: J1.10, TP30.1
- new net: J1.2, TP143.1
- new net: J1.21, TP152.1
- new net: J1.22, TP153.1
- new net: J1.3, TP144.1
- new net: J1.31, TP154.1
- new net: J1.32, TP155.1
- new net: J1.4, TP145.1
- new net: J1.5, TP146.1
- new net: J1.9, TP29.1
- new net: J8.8 (DEBUG-0), TP106.1
- new net C3-UART-RX: J1.38, J8.7 (CARD-RX)
- new net C3-UART-TX: J1.37, J8.6 (CARD-TX)
- new net CAN1_H: J1.33, J1.34
- new net CAN1_L: J1.35, J1.36
- new net CAN2_H: J1.17, J1.18
- new net CAN2_L: J1.19, J1.20
- new net GND: J1.27, J1.28, J1.29, J1.30, J3.SHLD, J4.SHLD, J7.4 (Pin_4), J8.14 (GND), J8.15 (PAD), J8.16 (PAD), J8.5 (GND)
- new net L_BAND_RF: J3.SIG
- new net OPD_PWR: J1.15, J1.16
- new net OPD_SCL: J1.13, J1.14
- new net OPD_SDA: J1.11, J1.12
- new net ORESAT_nSD: J1.39, J1.40
- new net OSD3358: SIP A/EEPROM_WP: J7.3 (Pin_3)
- new net OSD3358: SIP A/I2C0_SCL: J7.1 (Pin_1)
- new net OSD3358: SIP A/I2C0_SDA: J7.2 (Pin_2)
- new net OSD3358: SIP A/nRESET: R48.2
- new net PIN7-OUT: J1.7
- new net PIN8-OUT: J1.8
- new net UHF_BAND_RF: J4.SIG
- new net USB_CLI_DM: J8.4 (DEVICE-D-)
- new net USB_CLI_DP: J8.3 (DEVICE-D+)
- new net VBUS: J1.23, J1.24, J1.25, J1.26
- new net VIN_USB: J8.1 (VBUSP), J8.2 (VBUSP)
- new net nRESET: J8.10 (NRST), R48.1
- no-connect marks 0 -> 4
Other:
- removed sheet Connectors
- sheet L Band ports: added LBAND_IRQ, LBAND_LO_SCLK, LBAND_LO_SDATA, LBAND_LO_nLOCKED, LBAND_LO_nSEN, L_BAND_RF, SPI1_CS, SPI1_MISO, SPI1_MOSI, SPI1_SCLK; removed none
- sheet OPD and I2C Peripherals ports: added I2C2_SYS_DISABLE, I2C2_SYS_SCL, I2C2_SYS_SDA, OPD_CURRENT, OPD_PWR, OPD_SCL, OPD_SDA, OPD_nENABLE, OPD_nFAULT; removed none
- sheet OSD3358: SIP A ports: added EEPROM_WP, I2C0_SCL, I2C0_SDA, VIN_USB, nRESET; removed none
- sheet OSD3358: SIP B ports: added OPD_CURRENT, RADIO_CURRENT, UHF_FWD_RF_LOG, UHF_REV_RF_LOG, USB_CLI_DM, USB_CLI_DP, VIN_USB, nRESET; removed none
- sheet OSD3358: SIP C ports: added C3-UART-RX, C3-UART-TX, CAN1_H, CAN1_L, I2C2_SYS_DISABLE, I2C2_SYS_SCL, I2C2_SYS_SDA, LBAND_IRQ, L_BAND_ENABLE, OPD_nENABLE, OPD_nFAULT, PIN7-OUT, PIN8-OUT, RADIO_nFLT, SPI0_CS, SPI0_MISO, SPI0_MOSI, SPI0_SCLK, SPI1_CS, SPI1_MISO, SPI1_MOSI, SPI1_SCLK, UHF_ENABLE, UHF_IRQ, UHF_PA_ENABLE, UHF_TOT_CLEAR, UHF_TOT_OK; removed none
- sheet OSD3358: SIP D ports: added CAN2_H, CAN2_L, LBAND_LO_SCLK, LBAND_LO_SDATA, LBAND_LO_nLOCKED, LBAND_LO_nSEN, PET_WDT, RADIO_ENABLE; removed none
- sheet Power ports: added L_BAND_ENABLE, RADIO_CURRENT, RADIO_ENABLE, RADIO_nFLT, UHF_ENABLE; removed none
- sheet UHF Band ports: added SPI0_CS, SPI0_MISO, SPI0_MOSI, SPI0_SCLK, UHF_BAND_RF, UHF_FWD_RF_LOG, UHF_IRQ, UHF_PA_ENABLE, UHF_REV_RF_LOG, UHF_TOT_CLEAR, UHF_TOT_OK; removed none
- sheet Watchdog ports: added ORESAT_nSD, PET_WDT; removed none
- note added: "20 pin FFC Connector"
- note added: "Fiducials (Front)"
- note added: "Goes to Debug board; don't switch!"
- note added: "Mechanical"
- note added: "Needed for programming boot EEPROM TPS65217 I2C Addrs = 0x24 EEPROM I2C Addrs = 0x50 Needs 4 pos 1.27 mm socket and cable, e.g., Samtec SFSS-04-28-H-06.00-SR."
- note added: "Octavo reset!"
- note added: "OreSat Card Main Connector (Backplane v2)"
- note added: "Oresat Card Debug Connector"
- note added: "Oresat Card RF Connectors"
- note added: "Powers Octavo but *not* radios"
- note added: "SMPM Connectors to Backplane"
- note added: "USB Device (Ethernet over USB)"
